File: 01_Hardware/KiCad/Slave/Slave.kicad_sch (KiCad schematic)
At the start: 0 parts

Commit message: Slave KiCad 3D Draft
Parts:
- added J1, J3: Screw_Terminal_01x04, TerminalBlock_Phoenix:TerminalBlock_Phoenix_MKDS-3-4-5.08_1x04_P5.08mm_Horizontal, symbol Connector:Screw_Terminal_01x04
- added J2, J4: Conn_01x30_Female, Connector_PinSocket_2.54mm:PinSocket_1x30_P2.54mm_Vertical, symbol Connector:Conn_01x30_Female
- added Q1, Q2: AO3400A, Package_TO_SOT_SMD:SOT-23, symbol Transistor_FET:AO3400A
- added R1: 1k, Resistor_THT:R_Axial_DIN0204_L3.6mm_D1.6mm_P5.08mm_Horizontal, symbol Device:R
- added R2: 4k, Resistor_THT:R_Axial_DIN0204_L3.6mm_D1.6mm_P5.08mm_Horizontal, symbol Device:R
- added R3: 10k, Resistor_THT:R_Axial_DIN0204_L3.6mm_D1.6mm_P5.08mm_Horizontal, symbol Device:R
- added R4, R5: 400, Resistor_THT:R_Axial_DIN0204_L3.6mm_D1.6mm_P5.08mm_Horizontal, symbol Device:R
- added U1: LM393, Package_DIP:DIP-4_W7.62mm, symbol Comparator:LM393
Connections:
- new net: J2.24 (Pin_24), Q1.1 (G)
- new net: Q1.3 (D), R4.2
- new net: J2.27 (Pin_27), Q2.1 (G)
- new net: R1.2, R2.1, U1.2 (-)
- new net: J4.1 (Pin_1), R1.1
- new net: J4.11 (Pin_11), R3.2, U1.1
- new net: J4.2 (Pin_2), R3.1
- new net: Q2.3 (D), R5.2
- new net Bus: J1.4 (Pin_4), J3.1 (Pin_1), R4.1, R5.1, U1.3 (+)
- new net GND: J1.3 (Pin_3), J3.2 (Pin_2), J4.30 (Pin_30), Q1.2 (S), Q2.2 (S), R2.2
Other:
- company: HKa -> (none)
- title: DSI3 Master Tranceiver -> DSI3 Slave Tranceiver
