File: 01_Hardware/KiCad/Slave/_autosave-Slave.kicad_pcb (KiCad board)
At the start: 2 copper layers, 12 parts, among them J1 Screw_Terminal_01x04, J2 Conn_01x30_Female, J3 Screw_Terminal_01x04, J4 Conn_01x30_Female, Q1 AO3400A, Q2 AO3400A, U1 LM393

Commit message: Slave KiCad 3D Draft
Other:
- board text added: "Slave"
Changed lines of the file:
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@@
+    )
+  )
+  (gr_text "Slave" (at 172.72 136.525) (layer "F.Adhes")
+    (effects (font (size 5 5) (thickness 0.7)))
+  )
+  (zone (net 0) (net_name "") (layer "Edge.Cuts") (hatch edge 0.508)
+    (connect_pads (clearance 0.508))
+    (min_thickness 0.254)
+    (fill (thermal_gap 0.508) (thermal_bridge_width 0.508))
+    (polygon
+      (pts
+        (xy 206.375 150.495)
+        (xy 137.795 150.495)
+        (xy 137.795 56.515)
+        (xy 206.375 56.515)
+      )
     )
   )
